Commit message: fixed lidar not showing up

File: pi-code/src/jkl/description/ros2_control.xacro (robot description, xacro)
@@ -10,8 +10,8 @@
                 <param name="back_right_wheel_name">back_right_joint</param>
                 <param name="loop_rate">30</param>
-                <param name="device">/dev/serial/by-id/usb-Arduino__www.arduino.cc__Arduino_Mega_2560_12148509806232150650-if00</param>
+                <!-- <param name="device">/dev/serial/by-id/usb-Arduino__www.arduino.cc__Arduino_Mega_2560_12148509806232150650-if00</param> -->
                 <!-- <param name="device">/dev/serial/by-id/usb-Arduino_www.arduino.cc_0043_3433031323135101D081-if00</param> -->
-                <!-- <param name="device">/dev/serial/by-id/usb-STMicroelectronics_BLACKPILL_F401CC_CDC_in_FS_Mode_206734803156-if00</param> -->
-                <param name="baud_rate">115200</param>
+                <param name="device">/dev/serial/by-id/usb-STMicroelectronics_BLACKPILL_F401CC_CDC_in_FS_Mode_206734803156-if00</param>
+                <param name="baud_rate">57600</param>
                 <param name="timeout">1000</param>
                 <param name="enc_counts_per_rev">988</param>

File: pi-code/src/jkl/description/urdf/knight.xacro (robot description, xacro)
@@ -4,5 +4,16 @@
 <xacro:include filename="knight.trans" />
 <xacro:include filename="knight.gazebo" />
-<link name="base_link">
+<!-- BASE LINK -->
+    <link name="base_link">
+    </link>
+    <!-- BASE_FOOTPRINT LINK -->
+    <joint name="base_footprint_joint" type="fixed">
+        <parent link="base_link" />
+        <child link="base_footprint" />
+        <origin xyz="0 0 0" rpy="0 0 0" />
+    </joint>
+    <link name="base_footprint">
+    </link>
+<link name="chassis">
   <inertial>
     <origin xyz="-0.019247214224469626 -0.009218676459717027 -0.0016402160280328" rpy="0 0 0"/>
@@ -44,5 +55,5 @@
   </collision>
 </link>
-<link name="lidar_link">
+<link name="laser_frame">
   <inertial>
     <origin xyz="-0.00013026516237509694 0.000607970103502142 0.014307371775280256" rpy="0 0 0"/>
@@ -150,8 +161,13 @@
   <child link="camera_link"/>
 </joint>
+<joint name="chassis_joint" type="fixed">
+  <origin xyz="0.019247214224469626 0.009218676459717027 0.0016402160280328" rpy="0 0 0"/>
+  <parent link="base_link"/>
+  <child link="chassis"/>
+</joint>
 <joint name="lidar_joint" type="fixed">
   <origin xyz="0.044064 -0.006954 0.072354" rpy="0 0 0"/>
-  <parent link="base_link"/>
-  <child link="lidar_link"/>
+  <parent link="chassis"/>
+  <child link="laser_frame"/>
 </joint>
 <joint name="front_right_joint" type="continuous">
