Commit message: Mapping testing

File: pi-code/src/jkl/description/robot.urdf.xacro (robot description, xacro)
@@ -4,4 +4,5 @@
     <xacro:arg name="sim_mode" default="false"/>
     <xacro:include filename="urdf/simple.xacro" />
+    <!-- <xacro:include filename="urdf/knight.xacro" /> -->
     <xacro:if value="$(arg use_ros2_control)">
         <xacro:include filename="ros2_control.xacro" />

File: pi-code/src/jkl/description/urdf/knight.xacro (robot description, xacro)
@@ -24,5 +24,5 @@
     <origin xyz="0 0 0" rpy="0 0 0"/>
     <geometry>
-      <mesh filename="package://jkl/description/meshes/base_link.stl" scale="0.001 0.001 0.001"/>
+      <mesh filename="/home/g/Mobile_ML_Robot/pi-code/src/jkl/description/meshes/base_link.stl" scale="0.001 0.001 0.001"/>
     </geometry>
     <material name="silver"/>
@@ -31,5 +31,5 @@
     <origin xyz="0 0 0" rpy="0 0 0"/>
     <geometry>
-      <mesh filename="package://jkl/description/meshes/base_link.stl" scale="0.001 0.001 0.001"/>
+      <mesh filename="/home/g/Mobile_ML_Robot/pi-code/src/jkl/description/meshes/base_link.stl" scale="0.001 0.001 0.001"/>
     </geometry>
   </collision>
@@ -44,5 +44,5 @@
     <origin xyz="-0.110529 -0.039646 -0.024004" rpy="0 0 0"/>
     <geometry>
-      <mesh filename="package://jkl/description/meshes/camera_link.stl" scale="0.001 0.001 0.001"/>
+      <mesh filename="/home/g/Mobile_ML_Robot/pi-code/src/jkl/description/meshes/camera_link.stl" scale="0.001 0.001 0.001"/>
     </geometry>
     <material name="silver"/>
@@ -51,5 +51,5 @@
     <origin xyz="-0.110529 -0.039646 -0.024004" rpy="0 0 0"/>
     <geometry>
-      <mesh filename="package://jkl/description/meshes/camera_link.stl" scale="0.001 0.001 0.001"/>
+      <mesh filename="/home/g/Mobile_ML_Robot/pi-code/src/jkl/description/meshes/camera_link.stl" scale="0.001 0.001 0.001"/>
     </geometry>
   </collision>
@@ -64,5 +64,5 @@
     <origin xyz="-0.044064 0.006954 -0.072354" rpy="0 0 0"/>
     <geometry>
-      <mesh filename="package://jkl/description/meshes/lidar_link.stl" scale="0.001 0.001 0.001"/>
+      <mesh filename="/home/g/Mobile_ML_Robot/pi-code/src/jkl/description/meshes/lidar_link.stl" scale="0.001 0.001 0.001"/>
     </geometry>
     <material name="silver"/>
@@ -71,5 +71,5 @@
     <origin xyz="-0.044064 0.006954 -0.072354" rpy="0 0 0"/>
     <geometry>
-      <mesh filename="package://jkl/description/meshes/lidar_link.stl" scale="0.001 0.001 0.001"/>
+      <mesh filename="/home/g/Mobile_ML_Robot/pi-code/src/jkl/description/meshes/lidar_link.stl" scale="0.001 0.001 0.001"/>
     </geometry>
   </collision>
@@ -84,5 +84,5 @@
     <origin xyz="-0.035729 0.118178 0.032546" rpy="0 0 0"/>
     <geometry>
-      <mesh filename="package://jkl/description/meshes/front_right.stl" scale="0.001 0.001 0.001"/>
+      <mesh filename="/home/g/Mobile_ML_Robot/pi-code/src/jkl/description/meshes/front_right.stl" scale="0.001 0.001 0.001"/>
     </geometry>
     <material name="silver"/>
@@ -91,5 +91,5 @@
     <origin xyz="-0.035729 0.118178 0.032546" rpy="0 0 0"/>
     <geometry>
-      <mesh filename="package://jkl/description/meshes/front_right.stl" scale="0.001 0.001 0.001"/>
+      <mesh filename="/home/g/Mobile_ML_Robot/pi-code/src/jkl/description/meshes/front_right.stl" scale="0.001 0.001 0.001"/>
     </geometry>
   </collision>
@@ -104,5 +104,5 @@
     <origin xyz="0.104271 0.118178 0.032546" rpy="0 0 0"/>
     <geometry>
-      <mesh filename="package://jkl/description/meshes/back_right.stl" scale="0.001 0.001 0.001"/>
+      <mesh filename="/home/g/Mobile_ML_Robot/pi-code/src/jkl/description/meshes/back_right.stl" scale="0.001 0.001 0.001"/>
     </geometry>
     <material name="silver"/>
@@ -111,5 +111,5 @@
     <origin xyz="0.104271 0.118178 0.032546" rpy="0 0 0"/>
     <geometry>
-      <mesh filename="package://jkl/description/meshes/back_right.stl" scale="0.001 0.001 0.001"/>
+      <mesh filename="/home/g/Mobile_ML_Robot/pi-code/src/jkl/description/meshes/back_right.stl" scale="0.001 0.001 0.001"/>
     </geometry>
   </collision>
@@ -124,5 +124,5 @@
     <origin xyz="-0.035329 -0.104198 0.032546" rpy="0 0 0"/>
     <geometry>
-      <mesh filename="package://jkl/description/meshes/front_left.stl" scale="0.001 0.001 0.001"/>
+      <mesh filename="/home/g/Mobile_ML_Robot/pi-code/src/jkl/description/meshes/front_left.stl" scale="0.001 0.001 0.001"/>
     </geometry>
     <material name="silver"/>
@@ -131,5 +131,5 @@
     <origin xyz="-0.035329 -0.104198 0.032546" rpy="0 0 0"/>
     <geometry>
-      <mesh filename="package://jkl/description/meshes/front_left.stl" scale="0.001 0.001 0.001"/>
+      <mesh filename="/home/g/Mobile_ML_Robot/pi-code/src/jkl/description/meshes/front_left.stl" scale="0.001 0.001 0.001"/>
     </geometry>
   </collision>
@@ -144,5 +144,5 @@
     <origin xyz="0.104671 -0.104198 0.032546" rpy="0 0 0"/>
     <geometry>
-      <mesh filename="package://jkl/description/meshes/back_left.stl" scale="0.001 0.001 0.001"/>
+      <mesh filename="/home/g/Mobile_ML_Robot/pi-code/src/jkl/description/meshes/back_left.stl" scale="0.001 0.001 0.001"/>
     </geometry>
     <material name="silver"/>
@@ -151,5 +151,5 @@
     <origin xyz="0.104671 -0.104198 0.032546" rpy="0 0 0"/>
     <geometry>
-      <mesh filename="package://jkl/description/meshes/back_left.stl" scale="0.001 0.001 0.001"/>
+      <mesh filename="/home/g/Mobile_ML_Robot/pi-code/src/jkl/description/meshes/back_left.stl" scale="0.001 0.001 0.001"/>
     </geometry>
   </collision>

Commit message: .

File: pi-code/src/jkl/description/robot.urdf.xacro (robot description, xacro)
@@ -4,4 +4,5 @@
     <xacro:arg name="sim_mode" default="false"/>
     <xacro:include filename="urdf/simple.xacro" />
+     <!-- <xacro:include filename="urdf/knight.xacro" /> -->
     <xacro:if value="$(arg use_ros2_control)">
         <xacro:include filename="ros2_control.xacro" />

File: pi-code/src/jkl/description/urdf/simple.xacro (robot description, xacro)
@@ -30,6 +30,6 @@
     <xacro:property name="mu1" value="0.25" />
     <xacro:property name="mu2" value="0.25" />
-    <xacro:property name="sl1" value="5.0" />
-    <xacro:property name="sl2" value="5.0" />
+    <xacro:property name="sl1" value="10.0" />
+    <xacro:property name="sl2" value="10.0" />
     <material name="white">
         <color rgba="1 1 1 1" />
