Commit message: .

File: pi-code/src/jkl/description/gazebo_control.xacro (robot description, xacro)
@@ -1,31 +1,22 @@
 <?xml version="1.0"?>
 <robot xmlns:xacro="http://www.ros.org/wiki/xacro">
-  <gazebo>
-    <plugin name="gz::sim::systems::DiffDrive" filename="gz-sim-diff-drive-system">
-      <!-- Wheel Information -->
-      <front_left_joint>front_left_joint</front_left_joint>
-      <front_right_joint>front_right_joint</front_right_joint>
-      <back_left_joint>back_left_joint</back_left_joint>
-      <back_right_joint>back_right_joint</back_right_joint>
-      <wheel_separation>0.201</wheel_separation>
-      <wheel_radius>0.0425</wheel_radius>
-      <!-- Limits -->
-      <!-- <max_wheel_torque>200</max_wheel_torque> -->
-      <max_linear_acceleration>10</max_linear_acceleration>
-      <!-- Output -->
-      <frame_id>odom</frame_id>
-      <child_frame_id>base_link</child_frame_id>
-      <odom_topic>/odom</odom_topic>
-      <odom_publisher_frequency>30</odom_publisher_frequency>
-      <tf_topic>/tf</tf_topic>
-    </plugin>
-    <plugin filename="gz-sim-joint-state-publisher-system"
-            name="gz::sim::systems::JointStatePublisher">
-      <topic>joint_states</topic>
-      <joint_name>front_left_joint</joint_name>
-      <joint_name>front_right_joint</joint_name>
-      <joint_name>back_left_joint</joint_name>
-      <joint_name>back_right_joint</joint_name>
-    </plugin>
-  </gazebo>
+    <gazebo>
+        <plugin name="diff_drive" filename="libgazebo_ros_diff_drive.so">
+            <front_left_joint>front_left_joint</front_left_joint>
+            <front_right_joint>front_right_joint</front_right_joint>
+            <back_left_joint>back_left_joint</back_left_joint>
+            <back_right_joint>back_right_joint</back_right_joint>
+            <wheel_separation>0.201</wheel_separation>
+            <wheel_diameter>0.085</wheel_diameter>
+            <!-- Limits -->
+            <max_wheel_torque>200</max_wheel_torque>
+            <max_wheel_acceleration>10.0</max_wheel_acceleration>
+            <!-- Output -->
+            <odometry_frame>odom</odometry_frame>
+            <robot_base_frame>base_link</robot_base_frame>
+            <publish_odom>true</publish_odom>
+            <publish_odom_tf>true</publish_odom_tf>
+            <publish_wheel_tf>true</publish_wheel_tf>
+        </plugin>
+    </gazebo>
 </robot>

File: pi-code/src/jkl/description/ros2_control.xacro (robot description, xacro)
@@ -54,5 +54,5 @@
         <ros2_control name="GazeboSystem" type="system">
             <hardware>
-                <plugin>gz_ros2_control/GazeboSimSystem</plugin>
+                <plugin>gazebo_ros2_control/GazeboSystem</plugin>
             </hardware>
             <joint name="front_left_joint">
@@ -91,5 +91,5 @@
     </xacro:if>
     <gazebo>
-        <plugin name="gz_ros2_control::GazeboSimROS2ControlPlugin" filename="libgz_ros2_control-system.so">
+        <plugin name="gazebo_ros2_control" filename="libgazebo_ros2_control.so">
             <parameters>$(find jkl)/config/my_controllers.yaml</parameters>
             <parameters>$(find jkl)/config/gaz_ros2_ctl_use_sim.yaml</parameters>

File: pi-code/src/jkl/description/urdf/simple.xacro (robot description, xacro)
@@ -2,24 +2,24 @@
 <robot xmlns:xacro="http://www.ros.org/wiki/xacro" >
     <xacro:include filename="inertial_macros.xacro"/>
-    <xacro:property name="chassis_length" value="0.29"/>
-    <xacro:property name="chassis_width" value="0.265"/>
-    <xacro:property name="chassis_height" value="0.06"/>
+    <xacro:property name="chassis_length" value="0.290"/>
+    <xacro:property name="chassis_width" value="0.170"/>
+    <xacro:property name="chassis_height" value="0.036"/>
     <xacro:property name="head_length" value="${chassis_length/2}"/>
-    <xacro:property name="head_width" value="${chassis_width*1.2}"/>
-    <xacro:property name="head_height" value="${chassis_height}"/>
+    <xacro:property name="head_width" value="${chassis_width*1.4}"/>
+    <xacro:property name="head_height" value="0.0448"/>
     <xacro:property name="chassis_mass" value="1.0"/>
-    <xacro:property name="wheel_radius" value="0.045"/>
+    <xacro:property name="wheel_radius" value="0.0425"/>
     <xacro:property name="wheel_thickness" value="0.038"/>
     <xacro:property name="wheel_mass" value="0.05"/>
-    <xacro:property name="front_wheel_offset_x" value="0.226"/>
-    <xacro:property name="front_wheel_offset_y" value="0.1485"/>
-    <xacro:property name="front_wheel_offset_z" value="0.01"/>
-    <xacro:property name="caster_wheel_radius" value="0.01"/>
-    <xacro:property name="caster_wheel_mass" value="0.01"/>
-    <xacro:property name="back_wheel_offset_x" value="0.075"/>
+    <xacro:property name="front_wheel_offset_x" value="0.2148"/>
+    <xacro:property name="front_wheel_offset_y" value="${0.1024}"/>
+    <!-- <xacro:property name="front_wheel_offset_z" value="0.01"/> -->
+     <xacro:property name="front_wheel_offset_z" value="${wheel_radius}"/>
+    <xacro:property name="back_wheel_offset_x" value="0.0748"/>
     <xacro:property name="back_wheel_offset_y" value="${front_wheel_offset_y}"/>
-    <xacro:property name="back_wheel_offset_z" value="${front_wheel_offset_z - wheel_radius + caster_wheel_radius}"/>
-    <xacro:property name="lidar_offset_x" value="0.075"/>
-    <xacro:property name="lidar_offset_z" value="${chassis_height + head_height}"/>
+    <xacro:property name="back_wheel_offset_z" value="${front_wheel_offset_z}"/>
+    <xacro:property name="lidar_height" value="0.023"/>
+    <xacro:property name="lidar_offset_x" value="0.224"/>
+    <xacro:property name="lidar_offset_z" value="${chassis_height + head_height + front_wheel_offset_z}"/>
     <material name="white">
         <color rgba="1 1 1 1" />
@@ -56,5 +56,5 @@
     <link name="chassis">
         <visual>
-            <origin xyz="${chassis_length/2} 0 ${chassis_height/2}"/>
+            <origin xyz="${chassis_length/2} 0 ${chassis_height/2 + front_wheel_offset_z}"/>
             <geometry>
                 <box size="${chassis_length} ${chassis_width} ${chassis_height}"/>
@@ -63,5 +63,5 @@
         </visual>
         <collision>
-            <origin xyz="${chassis_length/2} 0 ${chassis_height/2}"/>
+            <origin xyz="${chassis_length/2} 0 ${chassis_height/2  + front_wheel_offset_z}"/>
             <geometry>
                 <box size="${chassis_length} ${chassis_width} ${chassis_height}"/>
@@ -69,5 +69,5 @@
         </collision>
         <xacro:inertial_box mass="0.5" x="${chassis_length}" y="${chassis_width}" z="${chassis_height}">
-            <origin xyz="${chassis_length/2} 0 ${chassis_height/2}" rpy="0 0 0"/>
+            <origin xyz="${chassis_length/2} 0 ${chassis_height/2  + front_wheel_offset_z}" rpy="0 0 0"/>
         </xacro:inertial_box>
     </link>
@@ -78,9 +78,9 @@
         <parent link="chassis"/>
         <child link="head"/>
-        <origin xyz="${-back_wheel_offset_x} 0 ${-front_wheel_offset_z}"/>
+        <origin xyz="${chassis_length - head_length/2} 0 ${head_height/2 + front_wheel_offset_z}"/>
     </joint>
     <link name="head">
         <visual>
-            <origin xyz="${front_wheel_offset_x + head_length/2} 0 ${head_height}"/>
+            <origin xyz="0 0 ${head_height}"/>
             <geometry>
                 <box size="${head_length} ${head_width} ${head_height}"/>
@@ -89,5 +89,5 @@
         </visual>
         <collision>
-            <origin xyz="${front_wheel_offset_x + head_length/2} 0 ${head_height}"/>
+            <origin xyz="0 0 ${head_height}"/>
             <geometry>
                 <box size="${head_length} ${head_width} ${head_height}"/>
@@ -95,5 +95,5 @@
         </collision>
         <xacro:inertial_box mass="0.5" x="${head_length}" y="${head_width}" z="${head_height}">
-            <origin xyz="${front_wheel_offset_x + head_length/2} 0 ${head_height}" rpy="0 0 0"/>
+            <origin xyz="0 0 ${head_height}" rpy="0 0 0"/>
         </xacro:inertial_box>
     </link>
@@ -104,5 +104,5 @@
         <parent link="base_link"/>
         <child link="front_left"/>
-        <origin xyz="${front_wheel_offset_x} ${front_wheel_offset_y} 0" rpy="-${pi/2} 0 0" />
+        <origin xyz="${front_wheel_offset_x - back_wheel_offset_x} ${front_wheel_offset_y} 0" rpy="-${pi/2} 0 0" />
         <axis xyz="0 0 1"/>
     </joint>
@@ -129,5 +129,5 @@
         <parent link="base_link"/>
         <child link="front_right"/>
-        <origin xyz="${front_wheel_offset_x} ${-front_wheel_offset_y} 0" rpy="${pi/2} 0 0" />
+        <origin xyz="${front_wheel_offset_x - back_wheel_offset_x} ${-front_wheel_offset_y} 0" rpy="${pi/2} 0 0" />
         <axis xyz="0 0 -1"/>
     </joint>
@@ -201,30 +201,59 @@
         <material>Gazebo/Blue</material>
     </gazebo>
-    <!-- CASTER WHEEL LINK -->
-    <joint name="caster_wheel_joint" type="fixed">
+    <joint name="lidar_joint" type="fixed">
         <parent link="chassis"/>
-        <child link="caster_wheel"/>
-        <origin xyz="${back_wheel_offset_x} 0 ${back_wheel_offset_z}"/>
-    </joint>
-    <link name="caster_wheel">
-        <visual>
-            <geometry>
-                <sphere radius="${caster_wheel_radius}"/>
+        <child link="laser_frame"/>
+        <origin xyz="${lidar_offset_x} 0 ${lidar_offset_z + 0.05}" rpy="0 0 0"/>
+    </joint>
+    <link name="laser_frame">
+        <visual>
+            <geometry>
+                <cylinder radius="0.05" length="${lidar_height}"/>
             </geometry>
             <material name="white"/>
         </visual>
-        <collision>
-            <geometry>
-                <sphere radius="${caster_wheel_radius}"/>
-            </geometry>
-        </collision>
-        <xacro:inertial_sphere mass="${caster_wheel_mass}" radius="${caster_wheel_radius}">
-            <origin xyz="0 0 0" rpy="0 0 0"/>
-        </xacro:inertial_sphere>
-    </link>
-    <gazebo reference="caster_wheel">
+        <visual>
+            <origin xyz="0 0 -0.05"/>
+            <geometry>
+                <cylinder radius="0.01" length="0.1"/>
+            </geometry>
+            <material name="white"/>
+        </visual>
+        <collision>
+            <geometry>
+                <cylinder radius="0.05" length="${lidar_height}"/>
+            </geometry>
+        </collision>
+        <xacro:inertial_cylinder mass="0.1" length="0.04" radius="0.05">
+            <origin xyz="0 0 0" rpy="0 0 0"/>
+        </xacro:inertial_cylinder>
+    </link>
+    <gazebo reference="laser_frame">
         <material>Gazebo/White</material>
-        <mu1 value="0.001"/>
-        <mu2 value="0.001"/>
+        <sensor name="laser" type="ray">
+            <pose> 0 0 0 0 0 0 </pose>
+            <visualize>false</visualize>
+            <update_rate>10</update_rate>
+            <ray>
+                <scan>
+                    <horizontal>
+                        <samples>360</samples>
+                        <min_angle>-3.14</min_angle>
+                        <max_angle>3.14</max_angle>
+                    </horizontal>
+                </scan>
+                <range>
+                    <min>0.3</min>
+                    <max>12</max>
+                </range>
+            </ray>
+            <plugin name="laser_controller" filename="libgazebo_ros_ray_sensor.so">
+                <ros>
+                    <argument>--ros-args --remap ~/out:=scan</argument>
+                </ros>
+                <output_type>sensor_msgs/LaserScan</output_type>
+                <frame_name>laser_frame</frame_name>
+            </plugin>
+        </sensor>
     </gazebo>
 </robot>

Commit message: color detection files

File: pi-code/src/jkl/description/gazebo_control.xacro (robot description, xacro)
@@ -4,13 +4,16 @@
     <plugin name="gz::sim::systems::DiffDrive" filename="gz-sim-diff-drive-system">
       <!-- Wheel Information -->
+      <num_wheel_pairs>2</num_wheel_pairs>
       <front_left_joint>front_left_joint</front_left_joint>
       <front_right_joint>front_right_joint</front_right_joint>
       <back_left_joint>back_left_joint</back_left_joint>
       <back_right_joint>back_right_joint</back_right_joint>
-      <wheel_separation>0.201</wheel_separation>
-      <wheel_radius>0.0425</wheel_radius>
+      <wheel_separation>0.35</wheel_separation>
+      <wheel_separation>0.35</wheel_separation>
+      <wheel_radius>0.0485</wheel_radius>
+      <wheel_radius>0.0485</wheel_radius>
       <!-- Limits -->
       <!-- <max_wheel_torque>200</max_wheel_torque> -->
-      <max_linear_acceleration>10</max_linear_acceleration>
+      <max_linear_acceleration>1.0</max_linear_acceleration>
       <!-- Output -->
       <frame_id>odom</frame_id>

File: pi-code/src/jkl/description/urdf/knight.xacro (robot description, xacro)
@@ -1,4 +1,5 @@
-<?xml version="1.0" ?>
+<?xml version="1.0"?>
 <robot name="knight" xmlns:xacro="http://www.ros.org/wiki/xacro">
+<<<<<<< Updated upstream
 <xacro:include filename="materials.xacro" />
 <xacro:include filename="knight.trans" />
@@ -195,3 +196,191 @@
   <axis xyz="0.0 1.0 -0.0"/>
 </joint>
+=======
+  <xacro:include filename="materials.xacro"/>
+  <xacro:include filename="knight.trans"/>
+  <xacro:include filename="knight.gazebo"/>
+  <!-- Define properties for wheels to reuse values -->
+  <xacro:property name="wheel_radius" value="0.0425"/>
+  <xacro:property name="wheel_thickness" value="0.036"/>
+  <!-- Root/base link -->
+  <link name="base_link">
+    <inertial>
+      <origin xyz="-0.019247214224469626 -0.009218676459717027 -0.0016402160280328" rpy="0 0 0"/>
+      <mass value="1.8335875472772791"/>
+      <inertia ixx="0.006149" iyy="0.014893" izz="0.017874" ixy="0.000425" iyz="6.7e-05" ixz="-0.000694"/>
+    </inertial>
+    <visual>
+      <origin xyz="0 0 0" rpy="0 0 0"/>
+      <geometry>
+        <mesh filename="package://jkl/description/meshes/base_link.stl" scale="0.001 0.001 0.001"/>
+      </geometry>
+      <material name="silver"/>
+    </visual>
+    <collision>
+      <origin xyz="0 0 0" rpy="0 0 0"/>
+      <geometry>
+        <mesh filename="package://jkl/description/meshes/base_link.stl" scale="0.001 0.001 0.001"/>
+      </geometry>
+    </collision>
+  </link>
+  <!-- Camera link if needed -->
+  <link name="camera_link">
+    <inertial>
+      <origin xyz="0.0022369050920157674 0.01190723740756753 -0.0106640979739921" rpy="0 0 0"/>
+      <mass value="0.0018917728244253016"/>
+      <inertia ixx="0.0" iyy="0.0" izz="0.0" ixy="0.0" iyz="0.0" ixz="-0.0"/>
+    </inertial>
+    <visual>
+      <origin xyz="-0.110529 -0.039646 -0.024004" rpy="0 0 0"/>
+      <geometry>
+        <mesh filename="package://jkl/description/meshes/camera_link.stl" scale="0.001 0.001 0.001"/>
+      </geometry>
+      <material name="silver"/>
+    </visual>
+    <collision>
+      <origin xyz="-0.110529 -0.039646 -0.024004" rpy="0 0 0"/>
+      <geometry>
+        <mesh filename="package://jkl/description/meshes/camera_link.stl" scale="0.001 0.001 0.001"/>
+      </geometry>
+    </collision>
+  </link>
+  <!-- Laser frame link if used -->
+  <link name="laser_frame">
+    <inertial>
+      <origin xyz="-0.00013026516237509694 0.000607970103502142 0.014307371775280256" rpy="0 0 0"/>
+      <mass value="0.007170751079753124"/>
+      <inertia ixx="3e-06" iyy="3e-06" izz="6e-06" ixy="-0.0" iyz="0.0" ixz="-0.0"/>
+    </inertial>
+    <visual>
+      <origin xyz="-0.044064 0.006954 -0.072354" rpy="0 0 0"/>
+      <geometry>
+        <mesh filename="package://jkl/description/meshes/lidar_link.stl" scale="0.001 0.001 0.001"/>
+      </geometry>
+      <material name="silver"/>
+    </visual>
+    <collision>
+      <origin xyz="-0.044064 0.006954 -0.072354" rpy="0 0 0"/>
+      <geometry>
+        <mesh filename="package://jkl/description/meshes/lidar_link.stl" scale="0.001 0.001 0.001"/>
+      </geometry>
+    </collision>
+  </link>
+  <!-- Wheel links -->
+  <link name="front_right">
+    <inertial>
+      <origin xyz="-1.5497830999564033e-06 0.003510779818395135 1.9940828647688202e-06" rpy="0 0 0"/>
+      <mass value="0.13957427599234848"/>
+      <inertia ixx="0.000102" iyy="0.000178" izz="0.000102" ixy="-0.0" iyz="0.0" ixz="-0.0"/>
+    </inertial>
+    <visual>
+      <origin xyz="-0.035729 0.118178 0.032546" rpy="0 1.5708 0"/>  <!-- rotated so cylinder’s axis matches wheel rolling axis -->
+      <geometry>
+        <cylinder radius="${wheel_radius}" length="${wheel_thickness}"/>
+      </geometry>
+      <material name="silver"/>
+    </visual>
+    <collision>
+      <origin xyz="-0.035729 0.118178 0.032546" rpy="0 1.5708 0"/>
+      <geometry>
+        <cylinder radius="${wheel_radius}" length="${wheel_thickness}"/>
+      </geometry>
+    </collision>
+  </link>
+  <link name="back_right">
+    <inertial>
+      <origin xyz="-1.5497830998106865e-06 0.0035107798183974387 1.994082864907598e-06" rpy="0 0 0"/>
+      <mass value="0.13957427599234848"/>
+      <inertia ixx="0.000102" iyy="0.000178" izz="0.000102" ixy="-0.0" iyz="0.0" ixz="-0.0"/>
+    </inertial>
+    <visual>
+      <origin xyz="0.104271 0.118178 0.032546" rpy="0 1.5708 0"/>
+      <geometry>
+        <cylinder radius="${wheel_radius}" length="${wheel_thickness}"/>
+      </geometry>
+      <material name="silver"/>
+    </visual>
+    <collision>
+      <origin xyz="0.104271 0.118178 0.032546" rpy="0 1.5708 0"/>
+      <geometry>
+        <cylinder radius="${wheel_radius}" length="${wheel_thickness}"/>
+      </geometry>
+    </collision>
+  </link>
+  <link name="front_left">
+    <inertial>
+      <origin xyz="-1.5493956658299557e-06 -0.00350998488597927 -1.4996934019281816e-06" rpy="0 0 0"/>
+      <mass value="0.13957427599234848"/>
+      <inertia ixx="0.000102" iyy="0.000178" izz="0.000102" ixy="0.0" iyz="0.0" ixz="0.0"/>
+    </inertial>
+    <visual>
+      <origin xyz="-0.035329 -0.104198 0.032546" rpy="0 1.5708 0"/>
+      <geometry>
+        <cylinder radius="${wheel_radius}" length="${wheel_thickness}"/>
+      </geometry>
+      <material name="silver"/>
+    </visual>
+    <collision>
+      <origin xyz="-0.035329 -0.104198 0.032546" rpy="0 1.5708 0"/>
+      <geometry>
+        <cylinder radius="${wheel_radius}" length="${wheel_thickness}"/>
+      </geometry>
+    </collision>
+  </link>
+  <link name="back_left">
+    <inertial>
+      <origin xyz="-1.5493956658646502e-06 -0.003509984885977299 -1.4996934019281816e-06" rpy="0 0 0"/>
+      <mass value="0.13957427599234848"/>
+      <inertia ixx="0.000102" iyy="0.000178" izz="0.000102" ixy="0.0" iyz="0.0" ixz="0.0"/>
+    </inertial>
+    <visual>
+      <origin xyz="0.104671 -0.104198 0.032546" rpy="0 1.5708 0"/>
+      <geometry>
+        <cylinder radius="${wheel_radius}" length="${wheel_thickness}"/>
+      </geometry>
+      <material name="silver"/>
+    </visual>
+    <collision>
+      <origin xyz="0.104671 -0.104198 0.032546" rpy="0 1.5708 0"/>
+      <geometry>
+        <cylinder radius="${wheel_radius}" length="${wheel_thickness}"/>
+      </geometry>
+    </collision>
+  </link>
+  <!-- Joints -->
+  <joint name="camera_joint" type="fixed">
+    <parent link="base_link"/>
+    <child link="camera_link"/>
+    <origin xyz="0.110529 0.039646 0.024004" rpy="0 0 0"/>
+  </joint>
+  <joint name="lidar_joint" type="fixed">
+    <parent link="base_link"/>
+    <child link="laser_frame"/>
+    <origin xyz="0.044064 -0.006954 0.072354" rpy="0 0 0"/>
+  </joint>
+  <!-- Wheel joints: define axis to match rolling (e.g. rotation about Y or X depending on geometry) -->
+  <joint name="front_right_joint" type="continuous">
+    <parent link="base_link"/>
+    <child link="front_right"/>
+    <origin xyz="-0.035729 0.118178 -0.032546" rpy="0 0 0"/>
+    <axis xyz="0 1 0"/> <!-- rotates around Y axis since cylinder oriented with rpy 0 1.5708 0 -->
+  </joint>
+  <joint name="back_right_joint" type="continuous">
+    <parent link="base_link"/>
+    <child link="back_right"/>
+    <origin xyz="0.104271 0.118178 -0.032546" rpy="0 0 0"/>
+    <axis xyz="0 1 0"/>
+  </joint>
+  <joint name="front_left_joint" type="continuous">
+    <parent link="base_link"/>
+    <child link="front_left"/>
+    <origin xyz="-0.035329 -0.104198 -0.032546" rpy="0 0 0"/>
+    <axis xyz="0 1 0"/>
+  </joint>
+  <joint name="back_left_joint" type="continuous">
+    <parent link="base_link"/>
+    <child link="back_left"/>
+    <origin xyz="0.104671 -0.104198 -0.032546" rpy="0 0 0"/>
+    <axis xyz="0 1 0"/>
+  </joint>
+>>>>>>> Stashed changes
 </robot>
