Commit message: making things run

File: pi-code/src/jkl/description/gazebo_control.xacro (robot description, xacro)
@@ -9,12 +9,6 @@
       <back_left_joint>back_left_joint</back_left_joint>
       <back_right_joint>back_right_joint</back_right_joint>
-<!-- <<<<<<< g
       <wheel_separation>0.207</wheel_separation>
-      <wheel_radius>0.085</wheel_radius>
-======= -->
-      <wheel_separation>0.35</wheel_separation>
-      <wheel_separation>0.35</wheel_separation>
-      <wheel_radius>0.0485</wheel_radius>
-      <wheel_radius>0.0485</wheel_radius>
+      <wheel_radius>0.0425</wheel_radius>
       <!-- Limits -->
       <!-- <max_wheel_torque>200</max_wheel_torque> -->

File: pi-code/src/jkl/description/ros2_control.xacro (robot description, xacro)
@@ -55,5 +55,5 @@
         <ros2_control name="GazeboSystem" type="system">
             <hardware>
-                <plugin>gazebo_ros2_control/GazeboSystem</plugin>
+                <plugin>gz_ros2_control/GazeboSimSystem</plugin>
             </hardware>
             <joint name="front_left_joint">
@@ -92,5 +92,5 @@
     </xacro:if>
     <gazebo>
-        <plugin name="gazebo_ros2_control" filename="libgazebo_ros2_control.so">
+        <plugin name="gz_ros2_control::GazeboSimROS2ControlPlugin" filename="libgz_ros2_control-system.so">
             <parameters>$(find jkl)/config/my_controllers.yaml</parameters>
             <parameters>$(find jkl)/config/gaz_ros2_ctl_use_sim.yaml</parameters>

File: pi-code/src/jkl/description/urdf/knight.xacro (robot description, xacro)
@@ -24,5 +24,5 @@
     <origin xyz="0 0 0" rpy="0 0 0"/>
     <geometry>
-      <mesh filename="/home/g/Mobile_ML_Robot/pi-code/src/jkl/description/meshes/base_link.stl" scale="0.001 0.001 0.001"/>
+      <mesh filename="package://jkl/description/meshes/base_link.stl" scale="0.001 0.001 0.001"/>
     </geometry>
     <material name="silver"/>
@@ -31,5 +31,5 @@
     <origin xyz="0 0 0" rpy="0 0 0"/>
     <geometry>
-      <mesh filename="/home/g/Mobile_ML_Robot/pi-code/src/jkl/description/meshes/base_link.stl" scale="0.001 0.001 0.001"/>
+      <mesh filename="package://jkl/description/meshes/base_link.stl" scale="0.001 0.001 0.001"/>
     </geometry>
   </collision>
@@ -44,5 +44,5 @@
     <origin xyz="-0.110529 -0.039646 -0.024004" rpy="0 0 0"/>
     <geometry>
-      <mesh filename="/home/g/Mobile_ML_Robot/pi-code/src/jkl/description/meshes/camera_link.stl" scale="0.001 0.001 0.001"/>
+      <mesh filename="package://jkl/description/meshes/camera_link.stl" scale="0.001 0.001 0.001"/>
     </geometry>
     <material name="silver"/>
@@ -51,5 +51,5 @@
     <origin xyz="-0.110529 -0.039646 -0.024004" rpy="0 0 0"/>
     <geometry>
-      <mesh filename="/home/g/Mobile_ML_Robot/pi-code/src/jkl/description/meshes/camera_link.stl" scale="0.001 0.001 0.001"/>
+      <mesh filename="package://jkl/description/meshes/camera_link.stl" scale="0.001 0.001 0.001"/>
     </geometry>
   </collision>
@@ -64,5 +64,5 @@
     <origin xyz="-0.044064 0.006954 -0.072354" rpy="0 0 0"/>
     <geometry>
-      <mesh filename="/home/g/Mobile_ML_Robot/pi-code/src/jkl/description/meshes/lidar_link.stl" scale="0.001 0.001 0.001"/>
+      <mesh filename="package://jkl/description/meshes/lidar_link.stl" scale="0.001 0.001 0.001"/>
     </geometry>
     <material name="silver"/>
@@ -71,5 +71,5 @@
     <origin xyz="-0.044064 0.006954 -0.072354" rpy="0 0 0"/>
     <geometry>
-      <mesh filename="/home/g/Mobile_ML_Robot/pi-code/src/jkl/description/meshes/lidar_link.stl" scale="0.001 0.001 0.001"/>
+      <mesh filename="package://jkl/description/meshes/lidar_link.stl" scale="0.001 0.001 0.001"/>
     </geometry>
   </collision>
@@ -84,5 +84,5 @@
     <origin xyz="-0.035729 0.118178 0.032546" rpy="0 0 0"/>
     <geometry>
-      <mesh filename="/home/g/Mobile_ML_Robot/pi-code/src/jkl/description/meshes/front_right.stl" scale="0.001 0.001 0.001"/>
+      <mesh filename="package://jkl/description/meshes/front_right.stl" scale="0.001 0.001 0.001"/>
     </geometry>
     <material name="silver"/>
@@ -91,5 +91,5 @@
     <origin xyz="-0.035729 0.118178 0.032546" rpy="0 0 0"/>
     <geometry>
-      <mesh filename="/home/g/Mobile_ML_Robot/pi-code/src/jkl/description/meshes/front_right.stl" scale="0.001 0.001 0.001"/>
+      <mesh filename="package://jkl/description/meshes/front_right.stl" scale="0.001 0.001 0.001"/>
     </geometry>
   </collision>
@@ -104,5 +104,5 @@
     <origin xyz="0.104271 0.118178 0.032546" rpy="0 0 0"/>
     <geometry>
-      <mesh filename="/home/g/Mobile_ML_Robot/pi-code/src/jkl/description/meshes/back_right.stl" scale="0.001 0.001 0.001"/>
+      <mesh filename="package://jkl/description/meshes/back_right.stl" scale="0.001 0.001 0.001"/>
     </geometry>
     <material name="silver"/>
@@ -111,5 +111,5 @@
     <origin xyz="0.104271 0.118178 0.032546" rpy="0 0 0"/>
     <geometry>
-      <mesh filename="/home/g/Mobile_ML_Robot/pi-code/src/jkl/description/meshes/back_right.stl" scale="0.001 0.001 0.001"/>
+      <mesh filename="package://jkl/description/meshes/back_right.stl" scale="0.001 0.001 0.001"/>
     </geometry>
   </collision>
@@ -124,5 +124,5 @@
     <origin xyz="-0.035329 -0.104198 0.032546" rpy="0 0 0"/>
     <geometry>
-      <mesh filename="/home/g/Mobile_ML_Robot/pi-code/src/jkl/description/meshes/front_left.stl" scale="0.001 0.001 0.001"/>
+      <mesh filename="package://jkl/description/meshes/front_left.stl" scale="0.001 0.001 0.001"/>
     </geometry>
     <material name="silver"/>
@@ -131,5 +131,5 @@
     <origin xyz="-0.035329 -0.104198 0.032546" rpy="0 0 0"/>
     <geometry>
-      <mesh filename="/home/g/Mobile_ML_Robot/pi-code/src/jkl/description/meshes/front_left.stl" scale="0.001 0.001 0.001"/>
+      <mesh filename="package://jkl/description/meshes/front_left.stl" scale="0.001 0.001 0.001"/>
     </geometry>
   </collision>
@@ -144,5 +144,5 @@
     <origin xyz="0.104671 -0.104198 0.032546" rpy="0 0 0"/>
     <geometry>
-      <mesh filename="/home/g/Mobile_ML_Robot/pi-code/src/jkl/description/meshes/back_left.stl" scale="0.001 0.001 0.001"/>
+      <mesh filename="package://jkl/description/meshes/back_left.stl" scale="0.001 0.001 0.001"/>
     </geometry>
     <material name="silver"/>
@@ -151,5 +151,5 @@
     <origin xyz="0.104671 -0.104198 0.032546" rpy="0 0 0"/>
     <geometry>
-      <mesh filename="/home/g/Mobile_ML_Robot/pi-code/src/jkl/description/meshes/back_left.stl" scale="0.001 0.001 0.001"/>
+      <mesh filename="package://jkl/description/meshes/back_left.stl" scale="0.001 0.001 0.001"/>
     </geometry>
   </collision>

File: pi-code/src/jkl/description/urdf/simple.xacro (robot description, xacro)
@@ -8,8 +8,6 @@
     <xacro:property name="head_width" value="${chassis_width*1.4}" />
     <xacro:property name="head_height" value="0.0448" />
-    <xacro:property name="chassis_mass" value="1.0" />
     <xacro:property name="wheel_radius" value="0.0425" />
     <xacro:property name="wheel_thickness" value="0.038" />
-    <xacro:property name="wheel_mass" value="0.05" />
     <xacro:property name="front_wheel_offset_x" value="0.2148" />
     <xacro:property name="front_wheel_offset_y" value="${0.1024}" />
@@ -28,4 +26,9 @@
     <xacro:property name="imu_offset_y" value="0.0" />
     <xacro:property name="imu_offset_z" value="${chassis_height + head_height + 0.02}" />
+    <xacro:property name="chassis_mass" value="1.0" />
+    <xacro:property name="lidar_mass" value="0.01" />
+    <xacro:property name="head_mass" value="0.01" />
+    <xacro:property name="imu_mass" value="0.001" />
+    <xacro:property name="wheel_mass" value="0.05" />
     <xacro:property name="mu1" value="0.25" />
     <xacro:property name="mu2" value="0.25" />
@@ -78,5 +81,5 @@
             </geometry>
         </collision>
-        <xacro:inertial_box mass="0.5" x="${chassis_length}" y="${chassis_width}"
+        <xacro:inertial_box mass="${chassis_mass}" x="${chassis_length}" y="${chassis_width}"
             z="${chassis_height}">
             <origin xyz="${chassis_length/2} 0 ${chassis_height/2  + front_wheel_offset_z}"
@@ -106,5 +109,5 @@
             </geometry>
         </collision>
-        <xacro:inertial_box mass="0.5" x="${head_length}" y="${head_width}" z="${head_height}">
+        <xacro:inertial_box mass="${head_mass}" x="${head_length}" y="${head_width}" z="${head_height}">
             <origin xyz="0 0 ${head_height}" rpy="0 0 0" />
         </xacro:inertial_box>
@@ -139,11 +142,11 @@
     <gazebo reference="front_left">
         <material>Gazebo/Red</material>
-        <mu1>${mu1}</mu1>        <!-- friction coefficient in one direction -->
-        <mu2>${mu2}</mu2>        <!-- friction coefficient in the perpendicular direction -->
-        <kp>1e5</kp>          <!-- contact stiffness -->
-        <kd>1.0</kd>          <!-- contact damping -->
-        <fdir1>1 0 0</fdir1>  <!-- primary friction direction -->
-        <slip1>${sl1}</slip1>    <!-- slip in primary direction -->
-        <slip2>${sl2}</slip2>    <!-- slip in perpendicular direction -->
+        <!-- <mu1>${mu1}</mu1>
+        <mu2>${mu2}</mu2>
+        <kp>1e5</kp>
+        <kd>1.0</kd>
+        <fdir1>1 0 0</fdir1>
+        <slip1>${sl1}</slip1>
+        <slip2>${sl2}</slip2>     -->
     </gazebo>
     <joint name="front_right_joint" type="continuous">
@@ -173,11 +176,11 @@
     <gazebo reference="front_right">
         <material>Gazebo/Red</material>
-        <mu1>${mu1}</mu1>        <!-- friction coefficient in one direction -->
-        <mu2>${mu2}</mu2>        <!-- friction coefficient in the perpendicular direction -->
-        <kp>1e5</kp>          <!-- contact stiffness -->
-        <kd>1.0</kd>          <!-- contact damping -->
-        <fdir1>1 0 0</fdir1>  <!-- primary friction direction -->
-        <slip1>${sl1}</slip1>    <!-- slip in primary direction -->
-        <slip2>${sl2}</slip2>    <!-- slip in perpendicular direction -->
+        <!-- <mu1>${mu1}</mu1>
+        <mu2>${mu2}</mu2>
+        <kp>1e5</kp>
+        <kd>1.0</kd>
+        <fdir1>1 0 0</fdir1>
+        <slip1>${sl1}</slip1>
+        <slip2>${sl2}</slip2>     -->
     </gazebo>
     <joint name="back_left_joint" type="continuous">
@@ -206,11 +209,11 @@
     <gazebo reference="back_left">
         <material>Gazebo/Blue</material>
-        <mu1>${mu1}</mu1>        <!-- friction coefficient in one direction -->
-        <mu2>${mu2}</mu2>        <!-- friction coefficient in the perpendicular direction -->
-        <kp>1e5</kp>          <!-- contact stiffness -->
-        <kd>1.0</kd>          <!-- contact damping -->
-        <fdir1>1 0 0</fdir1>  <!-- primary friction direction -->
-        <slip1>${sl1}</slip1>    <!-- slip in primary direction -->
-        <slip2>${sl2}</slip2>    <!-- slip in perpendicular direction -->
+        <!-- <mu1>${mu1}</mu1>
+        <mu2>${mu2}</mu2>
+        <kp>1e5</kp>
+        <kd>1.0</kd>
+        <fdir1>1 0 0</fdir1>
+        <slip1>${sl1}</slip1>
+        <slip2>${sl2}</slip2>     -->
     </gazebo>
     <joint name="back_right_joint" type="continuous">
@@ -239,11 +242,11 @@
     <gazebo reference="back_right">
         <material>Gazebo/Blue</material>
-        <mu1>${mu1}</mu1>        <!-- friction coefficient in one direction -->
-        <mu2>${mu2}</mu2>        <!-- friction coefficient in the perpendicular direction -->
-        <kp>1e5</kp>          <!-- contact stiffness -->
-        <kd>1.0</kd>          <!-- contact damping -->
-        <fdir1>1 0 0</fdir1>  <!-- primary friction direction -->
-        <slip1>${sl1}</slip1>    <!-- slip in primary direction -->
-        <slip2>${sl2}</slip2>    <!-- slip in perpendicular direction -->
+        <!-- <mu1>${mu1}</mu1>
+        <mu2>${mu2}</mu2>
+        <kp>1e5</kp>
+        <kd>1.0</kd>
+        <fdir1>1 0 0</fdir1>
+        <slip1>${sl1}</slip1>
+        <slip2>${sl2}</slip2>     -->
     </gazebo>
     <joint name="lidar_joint" type="fixed">
@@ -271,5 +274,5 @@
             </geometry>
         </collision>
-        <xacro:inertial_cylinder mass="0.1" length="0.04" radius="0.05">
+        <xacro:inertial_cylinder mass="${lidar_mass}" length="0.04" radius="0.05">
             <origin xyz="0 0 0" rpy="0 0 0" />
         </xacro:inertial_cylinder>
@@ -277,12 +280,14 @@
     <gazebo reference="laser_frame">
         <material>Gazebo/White</material>
-        <sensor name="laser" type="ray">
-            <pose> 0 0 0 0 0 0 </pose>
-            <visualize>false</visualize>
+        <sensor name="laser" type="gpu_lidar">
+            <pose relative_to='laser_frame'> 0 0 0 0 0 0 </pose>
+            <topic>scan</topic>
             <update_rate>10</update_rate>
-            <ray>
+            <gz_frame_id>laser_frame</gz_frame_id>
+            <lidar>
                 <scan>
                     <horizontal>
                         <samples>360</samples>
+                        <resolution>1</resolution>
                         <min_angle>-3.14</min_angle>
                         <max_angle>3.14</max_angle>
@@ -293,12 +298,7 @@
                     <max>12</max>
                 </range>
-            </ray>
-            <plugin name="laser_controller" filename="libgazebo_ros_ray_sensor.so">
-                <ros>
-                    <argument>~/out:=scan</argument>
-                </ros>
-                <output_type>sensor_msgs/LaserScan</output_type>
-                <frame_name>laser_frame</frame_name>
-            </plugin>
+             </lidar>
+            <always_on>true</always_on>
+            <visualize>true</visualize>
         </sensor>
     </gazebo>
@@ -325,5 +325,5 @@
             </geometry>
         </collision>
-        <xacro:inertial_box mass="0." x="${imu_length}" y="${imu_length}" z="0.01">
+        <xacro:inertial_box mass="${imu_mass}" x="${imu_length}" y="${imu_length}" z="0.01">
             <origin xyz="0 0 0" rpy="0 0 0" />
         </xacro:inertial_box>
@@ -332,17 +332,12 @@
         <material>Gazebo/White</material>
         <gravity>true</gravity>
-        <sensor name="my_imu" type="imu">
-            <!-- ensure the sensor is active (required) -->
+        <sensor name="imu_sensor" type="imu">
             <always_on>true</always_on>
             <update_rate>30</update_rate>
-            <visualize>true</visualize>
+            <visualize>false</visualize>
             <initialOrientationAsReference>true</initialOrientationAsReference>
             <!-- <gaussian_noise>0.001</gaussian_noise> -->
-            <plugin name="imu_controller" filename="libgazebo_ros_imu_sensor.so">
-                <ros>
-                    <namespace>/imu_broadcaster</namespace>
-                    <remapping>~/out:=imu</remapping>
-                </ros>
-            </plugin>
+            <topic>imu_broadcaster/imu</topic>
+            <gz_frame_id>imu_link</gz_frame_id>
         </sensor>
     </gazebo>
