Commit message: .

File: pi-code/src/jkl/description/urdf/simple.xacro (robot description, xacro)
@@ -1,39 +1,44 @@
 <?xml version="1.0"?>
-<robot xmlns:xacro="http://www.ros.org/wiki/xacro" >
-    <xacro:include filename="inertial_macros.xacro"/>
-    <xacro:property name="chassis_length" value="0.290"/>
-    <xacro:property name="chassis_width" value="0.170"/>
-    <xacro:property name="chassis_height" value="0.036"/>
-    <xacro:property name="head_length" value="${chassis_length/2}"/>
-    <xacro:property name="head_width" value="${chassis_width*1.4}"/>
-    <xacro:property name="head_height" value="0.0448"/>
-    <xacro:property name="chassis_mass" value="1.0"/>
-    <xacro:property name="wheel_radius" value="0.0425"/>
-    <xacro:property name="wheel_thickness" value="0.038"/>
-    <xacro:property name="wheel_mass" value="0.05"/>
-    <xacro:property name="front_wheel_offset_x" value="0.2148"/>
-    <xacro:property name="front_wheel_offset_y" value="${0.1024}"/>
+<robot xmlns:xacro="http://www.ros.org/wiki/xacro">
+    <xacro:include filename="inertial_macros.xacro" />
+    <xacro:property name="chassis_length" value="0.290" />
+    <xacro:property name="chassis_width" value="0.170" />
+    <xacro:property name="chassis_height" value="0.036" />
+    <xacro:property name="head_length" value="${chassis_length/2}" />
+    <xacro:property name="head_width" value="${chassis_width*1.4}" />
+    <xacro:property name="head_height" value="0.0448" />
+    <xacro:property name="chassis_mass" value="1.0" />
+    <xacro:property name="wheel_radius" value="0.0425" />
+    <xacro:property name="wheel_thickness" value="0.038" />
+    <xacro:property name="wheel_mass" value="0.05" />
+    <xacro:property name="front_wheel_offset_x" value="0.2148" />
+    <xacro:property name="front_wheel_offset_y" value="${0.1024}" />
     <!-- <xacro:property name="front_wheel_offset_z" value="0.01"/> -->
-     <xacro:property name="front_wheel_offset_z" value="${wheel_radius}"/>
-    <xacro:property name="back_wheel_offset_x" value="0.0748"/>
-    <xacro:property name="back_wheel_offset_y" value="${front_wheel_offset_y}"/>
-    <xacro:property name="back_wheel_offset_z" value="${front_wheel_offset_z}"/>
-    <xacro:property name="lidar_height" value="0.023"/>
-    <xacro:property name="lidar_offset_x" value="0.224"/>
-    <xacro:property name="lidar_offset_z" value="${chassis_height + head_height + front_wheel_offset_z}"/>
+    <xacro:property name="front_wheel_offset_z" value="${wheel_radius}" />
+    <xacro:property name="back_wheel_offset_x" value="0.0748" />
+    <xacro:property name="back_wheel_offset_y" value="${front_wheel_offset_y}" />
+    <xacro:property name="back_wheel_offset_z" value="${front_wheel_offset_z}" />
+    <xacro:property name="lidar_height" value="0.023" />
+    <xacro:property name="lidar_offset_x" value="0.224" />
+    <xacro:property name="lidar_offset_z"
+        value="${chassis_height + head_height + front_wheel_offset_z}" />
+    <xacro:property name="mu1" value="0.25" />
+    <xacro:property name="mu2" value="0.25" />
+    <xacro:property name="sl1" value="5.0" />
+    <xacro:property name="sl2" value="5.0" />
     <material name="white">
         <color rgba="1 1 1 1" />
     </material>
     <material name="orange">
-        <color rgba="1 0.3 0.1 1"/>
+        <color rgba="1 0.3 0.1 1" />
     </material>
     <material name="blue">
-        <color rgba="0.2 0.2 1 1"/>
+        <color rgba="0.2 0.2 1 1" />
     </material>
     <material name="black">
-        <color rgba="0 0 0 1"/>
+        <color rgba="0 0 0 1" />
     </material>
     <material name="red">
-        <color rgba="1 0 0 1"/>
+        <color rgba="1 0 0 1" />
     </material>
     <!-- BASE LINK -->
@@ -42,7 +47,7 @@
     <!-- BASE_FOOTPRINT LINK -->
     <joint name="base_footprint_joint" type="fixed">
-        <parent link="base_link"/>
-        <child link="base_footprint"/>
-        <origin xyz="0 0 0" rpy="0 0 0"/>
+        <parent link="base_link" />
+        <child link="base_footprint" />
+        <origin xyz="0 0 0" rpy="0 0 0" />
     </joint>
     <link name="base_footprint">
@@ -50,24 +55,26 @@
     <!-- CHASSIS LINK -->
     <joint name="chassis_joint" type="fixed">
-        <parent link="base_link"/>
-        <child link="chassis"/>
-        <origin xyz="${-back_wheel_offset_x} 0 ${-front_wheel_offset_z}"/>
+        <parent link="base_link" />
+        <child link="chassis" />
+        <origin xyz="${-back_wheel_offset_x} 0 ${-front_wheel_offset_z}" />
     </joint>
     <link name="chassis">
         <visual>
-            <origin xyz="${chassis_length/2} 0 ${chassis_height/2 + front_wheel_offset_z}"/>
-            <geometry>
-                <box size="${chassis_length} ${chassis_width} ${chassis_height}"/>
-            </geometry>
-            <material name="orange"/>
-        </visual>
-        <collision>
-            <origin xyz="${chassis_length/2} 0 ${chassis_height/2  + front_wheel_offset_z}"/>
-            <geometry>
-                <box size="${chassis_length} ${chassis_width} ${chassis_height}"/>
-            </geometry>
-        </collision>
-        <xacro:inertial_box mass="0.5" x="${chassis_length}" y="${chassis_width}" z="${chassis_height}">
-            <origin xyz="${chassis_length/2} 0 ${chassis_height/2  + front_wheel_offset_z}" rpy="0 0 0"/>
+            <origin xyz="${chassis_length/2} 0 ${chassis_height/2 + front_wheel_offset_z}" />
+            <geometry>
+                <box size="${chassis_length} ${chassis_width} ${chassis_height}" />
+            </geometry>
+            <material name="orange" />
+        </visual>
+        <collision>
+            <origin xyz="${chassis_length/2} 0 ${chassis_height/2  + front_wheel_offset_z}" />
+            <geometry>
+                <box size="${chassis_length} ${chassis_width} ${chassis_height}" />
+            </geometry>
+        </collision>
+        <xacro:inertial_box mass="0.5" x="${chassis_length}" y="${chassis_width}"
+            z="${chassis_height}">
+            <origin xyz="${chassis_length/2} 0 ${chassis_height/2  + front_wheel_offset_z}"
+                rpy="0 0 0" />
         </xacro:inertial_box>
     </link>
@@ -76,24 +83,24 @@
     </gazebo>
     <joint name="head_joint" type="fixed">
-        <parent link="chassis"/>
-        <child link="head"/>
-        <origin xyz="${chassis_length - head_length/2} 0 ${head_height/2 + front_wheel_offset_z}"/>
+        <parent link="chassis" />
+        <child link="head" />
+        <origin xyz="${chassis_length - head_length/2} 0 ${head_height/2 + front_wheel_offset_z}" />
     </joint>
     <link name="head">
         <visual>
-            <origin xyz="0 0 ${head_height}"/>
-            <geometry>
-                <box size="${head_length} ${head_width} ${head_height}"/>
-            </geometry>
-            <material name="black"/>
-        </visual>
-        <collision>
-            <origin xyz="0 0 ${head_height}"/>
-            <geometry>
-                <box size="${head_length} ${head_width} ${head_height}"/>
+            <origin xyz="0 0 ${head_height}" />
+            <geometry>
+                <box size="${head_length} ${head_width} ${head_height}" />
+            </geometry>
+            <material name="black" />
+        </visual>
+        <collision>
+            <origin xyz="0 0 ${head_height}" />
+            <geometry>
+                <box size="${head_length} ${head_width} ${head_height}" />
             </geometry>
         </collision>
         <xacro:inertial_box mass="0.5" x="${head_length}" y="${head_width}" z="${head_height}">
-            <origin xyz="0 0 ${head_height}" rpy="0 0 0"/>
+            <origin xyz="0 0 ${head_height}" rpy="0 0 0" />
         </xacro:inertial_box>
     </link>
@@ -102,129 +109,163 @@
     </gazebo>
     <joint name="front_left_joint" type="continuous">
-        <parent link="base_link"/>
-        <child link="front_left"/>
-        <origin xyz="${front_wheel_offset_x - back_wheel_offset_x} ${front_wheel_offset_y} 0" rpy="-${pi/2} 0 0" />
-        <axis xyz="0 0 1"/>
+        <parent link="base_link" />
+        <child link="front_left" />
+        <origin xyz="${front_wheel_offset_x - back_wheel_offset_x} ${front_wheel_offset_y} 0"
+            rpy="-${pi/2} 0 0" />
+        <axis xyz="0 0 1" />
     </joint>
     <link name="front_left">
         <visual>
             <geometry>
-                <cylinder radius="${wheel_radius}" length="${wheel_thickness}"/>
-            </geometry>
-            <material name="red"/>
-        </visual>
-        <collision>
-            <geometry>
-                <sphere radius="${wheel_radius}"/>
-            </geometry>
-        </collision>
-        <xacro:inertial_cylinder mass="${wheel_mass}" length="${wheel_thickness}" radius="${wheel_radius}">
-            <origin xyz="0 0 0" rpy="0 0 0"/>
+                <cylinder radius="${wheel_radius}" length="${wheel_thickness}" />
+            </geometry>
+            <material name="red" />
+        </visual>
+        <collision>
+            <geometry>
+                <sphere radius="${wheel_radius}" />
+            </geometry>
+        </collision>
+        <xacro:inertial_cylinder mass="${wheel_mass}" length="${wheel_thickness}"
+            radius="${wheel_radius}">
+            <origin xyz="0 0 0" rpy="0 0 0" />
         </xacro:inertial_cylinder>
     </link>
     <gazebo reference="front_left">
         <material>Gazebo/Red</material>
+        <mu1>${mu1}</mu1>        <!-- friction coefficient in one direction -->
+        <mu2>${mu2}</mu2>        <!-- friction coefficient in the perpendicular direction -->
+        <kp>1e5</kp>          <!-- contact stiffness -->
+        <kd>1.0</kd>          <!-- contact damping -->
+        <fdir1>1 0 0</fdir1>  <!-- primary friction direction -->
+        <slip1>${sl1}</slip1>    <!-- slip in primary direction -->
+        <slip2>${sl2}</slip2>    <!-- slip in perpendicular direction -->
     </gazebo>
     <joint name="front_right_joint" type="continuous">
-        <parent link="base_link"/>
-        <child link="front_right"/>
-        <origin xyz="${front_wheel_offset_x - back_wheel_offset_x} ${-front_wheel_offset_y} 0" rpy="${pi/2} 0 0" />
-        <axis xyz="0 0 -1"/>
+        <parent link="base_link" />
+        <child link="front_right" />
+        <origin xyz="${front_wheel_offset_x - back_wheel_offset_x} ${-front_wheel_offset_y} 0"
+            rpy="${pi/2} 0 0" />
+        <axis xyz="0 0 -1" />
     </joint>
     <link name="front_right">
         <visual>
             <geometry>
-                <cylinder radius="${wheel_radius}" length="${wheel_thickness}"/>
-            </geometry>
-            <material name="red"/>
-        </visual>
-        <collision>
-            <geometry>
-                <sphere radius="${wheel_radius}"/>
-            </geometry>
-        </collision>
-        <xacro:inertial_cylinder mass="${wheel_mass}" length="${wheel_thickness}" radius="${wheel_radius}">
-            <origin xyz="0 0 0" rpy="0 0 0"/>
+                <cylinder radius="${wheel_radius}" length="${wheel_thickness}" />
+            </geometry>
+            <material name="red" />
+        </visual>
+        <collision>
+            <geometry>
+                <sphere radius="${wheel_radius}" />
+            </geometry>
+        </collision>
+        <xacro:inertial_cylinder mass="${wheel_mass}" length="${wheel_thickness}"
+            radius="${wheel_radius}">
+            <origin xyz="0 0 0" rpy="0 0 0" />
         </xacro:inertial_cylinder>
     </link>
     <gazebo reference="front_right">
         <material>Gazebo/Red</material>
+        <mu1>${mu1}</mu1>        <!-- friction coefficient in one direction -->
+        <mu2>${mu2}</mu2>        <!-- friction coefficient in the perpendicular direction -->
+        <kp>1e5</kp>          <!-- contact stiffness -->
+        <kd>1.0</kd>          <!-- contact damping -->
+        <fdir1>1 0 0</fdir1>  <!-- primary friction direction -->
+        <slip1>${sl1}</slip1>    <!-- slip in primary direction -->
+        <slip2>${sl2}</slip2>    <!-- slip in perpendicular direction -->
     </gazebo>
     <joint name="back_left_joint" type="continuous">
-        <parent link="base_link"/>
-        <child link="back_left"/>
+        <parent link="base_link" />
+        <child link="back_left" />
         <origin xyz="0 ${back_wheel_offset_y} 0" rpy="-${pi/2} 0 0" />
-        <axis xyz="0 0 1"/>
+        <axis xyz="0 0 1" />
     </joint>
     <link name="back_left">
         <visual>
             <geometry>
-                <cylinder radius="${wheel_radius}" length="${wheel_thickness}"/>
-            </geometry>
-            <material name="blue"/>
-        </visual>
-        <collision>
-            <geometry>
-                <sphere radius="${wheel_radius}"/>
-            </geometry>
-        </collision>
-        <xacro:inertial_cylinder mass="${wheel_mass}" length="${wheel_thickness}" radius="${wheel_radius}">
-            <origin xyz="0 0 0" rpy="0 0 0"/>
+                <cylinder radius="${wheel_radius}" length="${wheel_thickness}" />
+            </geometry>
+            <material name="blue" />
+        </visual>
+        <collision>
+            <geometry>
+                <sphere radius="${wheel_radius}" />
+            </geometry>
+        </collision>
+        <xacro:inertial_cylinder mass="${wheel_mass}" length="${wheel_thickness}"
+            radius="${wheel_radius}">
+            <origin xyz="0 0 0" rpy="0 0 0" />
         </xacro:inertial_cylinder>
     </link>
     <gazebo reference="back_left">
         <material>Gazebo/Blue</material>
+        <mu1>${mu1}</mu1>        <!-- friction coefficient in one direction -->
+        <mu2>${mu2}</mu2>        <!-- friction coefficient in the perpendicular direction -->
+        <kp>1e5</kp>          <!-- contact stiffness -->
+        <kd>1.0</kd>          <!-- contact damping -->
+        <fdir1>1 0 0</fdir1>  <!-- primary friction direction -->
+        <slip1>${sl1}</slip1>    <!-- slip in primary direction -->
+        <slip2>${sl2}</slip2>    <!-- slip in perpendicular direction -->
     </gazebo>
     <joint name="back_right_joint" type="continuous">
-        <parent link="base_link"/>
-        <child link="back_right"/>
+        <parent link="base_link" />
+        <child link="back_right" />
         <origin xyz="0 ${-back_wheel_offset_y} 0" rpy="${pi/2} 0 0" />
-        <axis xyz="0 0 -1"/>
+        <axis xyz="0 0 -1" />
     </joint>
     <link name="back_right">
         <visual>
             <geometry>
-                <cylinder radius="${wheel_radius}" length="${wheel_thickness}"/>
-            </geometry>
-            <material name="blue"/>
-        </visual>
-        <collision>
-            <geometry>
-                <sphere radius="${wheel_radius}"/>
-            </geometry>
-        </collision>
-        <xacro:inertial_cylinder mass="${wheel_mass}" length="${wheel_thickness}" radius="${wheel_radius}">
-            <origin xyz="0 0 0" rpy="0 0 0"/>
+                <cylinder radius="${wheel_radius}" length="${wheel_thickness}" />
+            </geometry>
+            <material name="blue" />
+        </visual>
+        <collision>
+            <geometry>
+                <sphere radius="${wheel_radius}" />
+            </geometry>
+        </collision>
+        <xacro:inertial_cylinder mass="${wheel_mass}" length="${wheel_thickness}"
+            radius="${wheel_radius}">
+            <origin xyz="0 0 0" rpy="0 0 0" />
         </xacro:inertial_cylinder>
     </link>
     <gazebo reference="back_right">
         <material>Gazebo/Blue</material>
+        <mu1>${mu1}</mu1>        <!-- friction coefficient in one direction -->
+        <mu2>${mu2}</mu2>        <!-- friction coefficient in the perpendicular direction -->
+        <kp>1e5</kp>          <!-- contact stiffness -->
+        <kd>1.0</kd>          <!-- contact damping -->
+        <fdir1>1 0 0</fdir1>  <!-- primary friction direction -->
+        <slip1>${sl1}</slip1>    <!-- slip in primary direction -->
+        <slip2>${sl2}</slip2>    <!-- slip in perpendicular direction -->
     </gazebo>
     <joint name="lidar_joint" type="fixed">
-        <parent link="chassis"/>
-        <child link="laser_frame"/>
-        <origin xyz="${lidar_offset_x} 0 ${lidar_offset_z + 0.05}" rpy="0 0 0"/>
+        <parent link="chassis" />
+        <child link="laser_frame" />
+        <origin xyz="${lidar_offset_x} 0 ${lidar_offset_z + 0.05}" rpy="0 0 0" />
     </joint>
     <link name="laser_frame">
         <visual>
             <geometry>
-                <cylinder radius="0.05" length="${lidar_height}"/>
-            </geometry>
-            <material name="white"/>
-        </visual>
-        <visual>
-            <origin xyz="0 0 -0.05"/>
-            <geometry>
-                <cylinder radius="0.01" length="0.1"/>
-            </geometry>
-            <material name="white"/>
-        </visual>
-        <collision>
-            <geometry>
-                <cylinder radius="0.05" length="${lidar_height}"/>
+                <cylinder radius="0.05" length="${lidar_height}" />
+            </geometry>
+            <material name="white" />
+        </visual>
+        <visual>
+            <origin xyz="0 0 -0.05" />
+            <geometry>
+                <cylinder radius="0.01" length="0.1" />
+            </geometry>
+            <material name="white" />
+        </visual>
+        <collision>
+            <geometry>
+                <cylinder radius="0.05" length="${lidar_height}" />
             </geometry>
         </collision>
         <xacro:inertial_cylinder mass="0.1" length="0.04" radius="0.05">
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
Commit message: adding imu

File: pi-code/src/jkl/description/urdf/simple.xacro (robot description, xacro)
@@ -23,4 +23,9 @@
     <xacro:property name="lidar_offset_z"
         value="${chassis_height + head_height + front_wheel_offset_z}" />
+    <xacro:property name="imu_length" value="0.030" />
+    <xacro:property name="imu_width" value="0.015" />
+    <xacro:property name="imu_offset_x" value="${chassis_length}" />
+    <xacro:property name="imu_offset_y" value="0.0" />
+    <xacro:property name="imu_offset_z" value="${chassis_height + head_height + 0.02}" />
     <xacro:property name="mu1" value="0.25" />
     <xacro:property name="mu2" value="0.25" />
@@ -298,3 +303,45 @@
         </sensor>
     </gazebo>
+    <joint name="imu_joint" type="fixed">
+        <parent link="chassis" />
+        <child link="imu_link" />
+        <origin xyz="${imu_offset_x} ${imu_offset_y} ${imu_offset_z}" rpy="0 0 0" />
+    </joint>
+    <link name="imu_link">
+        <visual>
+            <geometry>
+                <box size="${imu_length} ${imu_width} 0.01" />
+            </geometry>
+            <material name="white" />
+        </visual>
+        <visual>
+            <geometry>
+                <box size="${imu_length} ${imu_width} 0.01" />
+            </geometry>
+        </visual>
+        <collision>
+            <geometry>
+                <box size="${imu_length} ${imu_width} 0.01" />
+            </geometry>
+        </collision>
+        <xacro:inertial_box mass="0." x="${imu_length}" y="${imu_length}" z="0.01">
+            <origin xyz="0 0 0" rpy="0 0 0" />
+        </xacro:inertial_box>
+    </link>
+    <gazebo reference="imu_link">
+        <material>Gazebo/White</material>
+        <sensor name="my_imu" type="imu">
+            <!-- ensure the sensor is active (required) -->
+            <always_on>true</always_on>
+            <update_rate>30</update_rate>
+            <!-- <gaussian_noise>0.001</gaussian_noise> -->
+            <plugin name="imu_controller" filename="libgazebo_ros_imu_sensor.so">
+                <ros>
+                    <!-- publish to /imu/data -->
+                    <namespace>/imu</namespace>
+                    <remapping>~/out:=data</remapping>
+                </ros>
+            </plugin>
+        </sensor>
+    </gazebo>
 </robot>

Commit message: .

File: pi-code/src/jkl/description/urdf/simple.xacro (robot description, xacro)
@@ -306,5 +306,5 @@
         <parent link="chassis" />
         <child link="imu_link" />
-        <origin xyz="${imu_offset_x} ${imu_offset_y} ${imu_offset_z}" rpy="0 0 0" />
+        <origin xyz="${imu_offset_x} ${imu_offset_y} ${imu_offset_z}" rpy="0 0 ${-pi/2}" />
     </joint>
     <link name="imu_link">
