Commit message: fixing robot_localization

File: pi-code/src/jkl/description/urdf/simple.xacro (robot description, xacro)
@@ -5,23 +5,21 @@
     <xacro:property name="chassis_width" value="0.170" />
     <xacro:property name="chassis_height" value="0.036" />
-    <xacro:property name="head_length" value="${chassis_length/2}" />
+    <xacro:property name="head_length" value="${chassis_length/2.5}" />
     <xacro:property name="head_width" value="${chassis_width*1.4}" />
     <xacro:property name="head_height" value="0.0448" />
     <xacro:property name="wheel_radius" value="0.0425" />
     <xacro:property name="wheel_thickness" value="0.038" />
-    <xacro:property name="front_wheel_offset_x" value="0.2148" />
+    <xacro:property name="front_wheel_offset_x" value="${0.125 - wheel_radius}" />
     <xacro:property name="front_wheel_offset_y" value="${0.1024}" />
-    <!-- <xacro:property name="front_wheel_offset_z" value="0.01"/> -->
     <xacro:property name="front_wheel_offset_z" value="${wheel_radius}" />
-    <xacro:property name="back_wheel_offset_x" value="0.0748" />
+    <xacro:property name="back_wheel_offset_x" value="${0.125 - wheel_radius}" />
     <xacro:property name="back_wheel_offset_y" value="${front_wheel_offset_y}" />
     <xacro:property name="back_wheel_offset_z" value="${front_wheel_offset_z}" />
     <xacro:property name="lidar_height" value="0.023" />
-    <xacro:property name="lidar_offset_x" value="0.224" />
-    <xacro:property name="lidar_offset_z"
-        value="${chassis_height + head_height + front_wheel_offset_z}" />
+    <xacro:property name="lidar_offset_x" value="${front_wheel_offset_x + 0.02}" />
+    <xacro:property name="lidar_offset_z" value="${chassis_height + head_height + front_wheel_offset_z}" />
     <xacro:property name="imu_length" value="0.030" />
     <xacro:property name="imu_width" value="0.015" />
-    <xacro:property name="imu_offset_x" value="${chassis_length}" />
+    <xacro:property name="imu_offset_x" value="${chassis_length/2}" />
     <xacro:property name="imu_offset_y" value="0.0" />
     <xacro:property name="imu_offset_z" value="${chassis_height + head_height + 0.02}" />
@@ -35,4 +33,5 @@
     <xacro:property name="sl1" value="10.0" />
     <xacro:property name="sl2" value="10.0" />
+    <xacro:property name="centre_of_rot_offset_x" value="${-0.02}" />
     <material name="white">
         <color rgba="1 1 1 1" />
@@ -65,9 +64,9 @@
         <parent link="base_link" />
         <child link="chassis" />
-        <origin xyz="${-back_wheel_offset_x} 0 ${-front_wheel_offset_z}" />
+        <origin xyz="${centre_of_rot_offset_x} 0 ${-front_wheel_offset_z}" />
     </joint>
     <link name="chassis">
         <visual>
-            <origin xyz="${chassis_length/2} 0 ${chassis_height/2 + front_wheel_offset_z}" />
+            <origin xyz="0 0 ${chassis_height/2 + front_wheel_offset_z}" />
             <geometry>
                 <box size="${chassis_length} ${chassis_width} ${chassis_height}" />
@@ -76,5 +75,5 @@
         </visual>
         <collision>
-            <origin xyz="${chassis_length/2} 0 ${chassis_height/2  + front_wheel_offset_z}" />
+            <origin xyz="0 0 ${chassis_height/2  + front_wheel_offset_z}" />
             <geometry>
                 <box size="${chassis_length} ${chassis_width} ${chassis_height}" />
@@ -83,5 +82,5 @@
         <xacro:inertial_box mass="${chassis_mass}" x="${chassis_length}" y="${chassis_width}"
             z="${chassis_height}">
-            <origin xyz="${chassis_length/2} 0 ${chassis_height/2  + front_wheel_offset_z}"
+            <origin xyz="0 0 ${chassis_height/2  + front_wheel_offset_z}"
                 rpy="0 0 0" />
         </xacro:inertial_box>
@@ -93,5 +92,5 @@
         <parent link="chassis" />
         <child link="head" />
-        <origin xyz="${chassis_length - head_length/2} 0 ${head_height/2 + front_wheel_offset_z}" />
+        <origin xyz="${chassis_length/2 - head_length/2} 0 ${head_height/2 + front_wheel_offset_z}" />
     </joint>
     <link name="head">
@@ -119,5 +118,5 @@
         <parent link="base_link" />
         <child link="front_left" />
-        <origin xyz="${front_wheel_offset_x - back_wheel_offset_x} ${front_wheel_offset_y} 0"
+        <origin xyz="${front_wheel_offset_x + centre_of_rot_offset_x} ${front_wheel_offset_y} 0"
             rpy="-${pi/2} 0 0" />
         <axis xyz="0 0 1" />
@@ -153,5 +152,5 @@
         <parent link="base_link" />
         <child link="front_right" />
-        <origin xyz="${front_wheel_offset_x - back_wheel_offset_x} ${-front_wheel_offset_y} 0"
+        <origin xyz="${front_wheel_offset_x + centre_of_rot_offset_x} ${-front_wheel_offset_y} 0"
             rpy="${pi/2} 0 0" />
         <axis xyz="0 0 -1" />
@@ -187,5 +186,5 @@
         <parent link="base_link" />
         <child link="back_left" />
-        <origin xyz="0 ${back_wheel_offset_y} 0" rpy="-${pi/2} 0 0" />
+        <origin xyz="${-back_wheel_offset_x + centre_of_rot_offset_x} ${back_wheel_offset_y} 0" rpy="-${pi/2} 0 0" />
         <axis xyz="0 0 1" />
     </joint>
@@ -220,5 +219,5 @@
         <parent link="base_link" />
         <child link="back_right" />
-        <origin xyz="0 ${-back_wheel_offset_y} 0" rpy="${pi/2} 0 0" />
+        <origin xyz="${-back_wheel_offset_x + centre_of_rot_offset_x} ${-back_wheel_offset_y} 0" rpy="${pi/2} 0 0" />
         <axis xyz="0 0 -1" />
     </joint>

Commit message: fixed robot odom drift along Y axis

File: pi-code/src/jkl/description/urdf/simple.xacro (robot description, xacro)
@@ -21,5 +21,5 @@
     <xacro:property name="imu_length" value="0.030" />
     <xacro:property name="imu_width" value="0.015" />
-    <xacro:property name="imu_offset_x" value="${chassis_length/2}" />
+    <xacro:property name="imu_offset_x" value="${front_wheel_offset_x + centre_of_rot_offset_x + imu_length/2 + 0.04}" />
     <xacro:property name="imu_offset_y" value="0.0" />
     <xacro:property name="imu_offset_z" value="${chassis_height + head_height + 0.02}" />
